Commit message: Lesson 2: Project Go Chase It: Change to Publisher Subscriber Class and Custom Robot
Lesson 2: Project Go Chase It: Move global logic into class contained code

Lesson 2: Project Go Chase It: Remove robot from world

Lesson 2: Project Go Chase It: Modified Robot Design

Update .gitignore to ignore .catkin_workspace and .vscode

Project 2: Project Go Chase It: clean up files

File: lesson02_ros/project-go-chase-it/src/my_robot/urdf/my_robot.xacro (robot description, xacro)
@@ -38,5 +38,5 @@
 		<visual name="back_caster_visual">
 			<origin xyz="-0.15 0 -0.05" rpy=" 0 0 0" />
-			<geometry>
+		<geometry>
 				<sphere radius="0.05" />
 			</geometry>
@@ -55,4 +55,52 @@
 		</visual>
 	</link>
+	<joint type="fixed" name="chassis_body_joint">
+		<origin xyz="0 0 0.1" rpy="0 0 0" />
+		<parent link="chassis" />
+		<child link="chassis_body" />
+	</joint>
+	<link name="chassis_body">
+		<visual>
+			<origin xyz="0 0 0" rpy="0 0 0" />
+			<geometry>
+				<box size="0.2 0.2 0.1" />
+			</geometry>
+		</visual>
+		<collision>
+			<origin xyz="0 0 0" rpy="0 0 0" />
+			<geometry>
+				<box size="0.2 0.2 0.1" />
+			</geometry>
+		</collision>
+		<intertial>
+			<mass value="5.0" />
+			<origin xyz="0 0 0" rpy=" 0 0 0" />
+			<inertia ixx="0.1" ixy="0" ixz="0" iyy="0.1" iyz="0" izz="0.1" />
+		</intertial>
+	</link>
+	<joint type="fixed" name="chassis_roof_joint">
+		<origin xyz="0 0 0.15" rpy="0 0 0" />
+		<parent link="chassis" />
+		<child link="chassis_roof" />
+	</joint>
+	<link name="chassis_roof">
+		<visual>
+			<origin xyz="0 0 0" rpy="0 0 0" />
+			<geometry>
+				<sphere radius="0.1" />
+			</geometry>
+		</visual>
+		<collision>
+			<origin xyz="0 0 0" rpy="0 0 0" />
+			<geometry>
+				<sphere radius="0.1" />
+			</geometry>
+		</collision>
+		<inertial>
+			<mass value="2.0" />
+			<origin xyz="0 0 0" rpy=" 0 0 0" />
+			<inertia ixx="0.1" ixy="0" ixz="0" iyy="0.1" iyz="0" izz="0.1" />
+		</inertial>
+	</link>
 	<joint type="continuous" name="left_wheel_hinge">
 		<origin xyz="0 0.15 0" rpy="0 0 0" />
@@ -110,5 +158,5 @@
 	</link>
 	<joint type="fixed" name="camera_joint">
-		<origin xyz="0.2 0 0" rpy="0 0 0" />
+		<origin xyz="0.1 0 0.15" rpy="0 0 0" />
 		<parent link="chassis" />
 		<child link="camera" />
@@ -135,5 +183,5 @@
 	</link>
 	<joint type="fixed" name="hokuyo_joint">
-		<origin xyz="0.15 0 0.1" rpy="0 0 0" />
+		<origin xyz="0 0 0.25" rpy="0 0 0" />
 		<parent link="chassis" />
 		<child link="hokuyo" />
@@ -161,20 +209,30 @@
 	<gazebo reference="left_wheel">
 		<material>
-			Gazebo/Green
+			Gazebo/Orange
 		</material>
 	</gazebo>
 	<gazebo reference="right_wheel">
 		<material>
-			Gazebo/Green
+			Gazebo/Orange
 		</material>
 	</gazebo>
 	<gazebo reference="camera">
 		<material>
-			Gazebo/Red
+			Gazebo/White
 		</material>
 	</gazebo>
 	<gazebo reference="chassis">
 		<material>
-			Gazebo/Blue
+			Gazebo/Yellow
+		</material>
+	</gazebo>
+	<gazebo reference="chassis_body">
+		<material>
+			Gazebo/Yellow
+		</material>
+	</gazebo>
+	<gazebo reference="chassis_roof">
+		<material>
+			Gazebo/Yellow
 		</material>
 	</gazebo>
